File: dds-sweeper-board/dds-sweeper-board.kicad_pcb (KiCad board)
At the start: 2 copper layers, 56 x 65 mm, 10 parts, among them J1 REF CLK, J2 3V3, J3 1V8, J4 Headers for AD9959 Eval Board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, J5 Trigger In, SW1 Pico Power Switch, U1 Pico, U3 5V->1V8 Linear Regulator

Commit message: Updated board design
Parts:
- removed J2: 3V3, Connector_Coaxial:SMA_Samtec_SMA-J-P-X-ST-EM1_EdgeMount
- removed SW1: Pico Power Switch, Connector_PinSocket_2.54mm:PinSocket_1x03_P2.54mm_Vertical
- added C3: 0.1uF, Capacitor_SMD:C_0805_2012Metric_Pad1.18x1.45mm_HandSolder, F.Cu at (40.8, 76.2)
- added C4: 0.1uF, Capacitor_SMD:C_0805_2012Metric_Pad1.18x1.45mm_HandSolder, F.Cu at (35.7, 85.7)
- added J6: RESET, Connector_PinSocket_2.54mm:PinSocket_1x03_P2.54mm_Vertical, F.Cu at (40.9, 71.0)
- added J7: DDS PWR, Connector_PinSocket_2.54mm:PinSocket_1x03_P2.54mm_Vertical, F.Cu at (35.7, 81.4)
- C1: value 1uF -> 0.1uF
- J1: value REF CLK -> REF CLK OUT
- J4: value Headers for AD9959 Eval Board U2 -> AD9959 Eval Header; footprint Custom_Conn:PinSocket_2x16_P2.54mm_Vertical_DDS_Sweeper -> Connector_PinSocket_2.54mm:PinSocket_2x16_P2.54mm_Vertical
- U3: value 5V->1V8 Linear Regulator -> XC6210B18
- moved J5 76.8 mm to (34.1, 37.7), turned to -90 degrees
- moved J3 76.3 mm to (34.1, 94.6), turned to -90 degrees
- moved C2 64.5 mm to (35.7, 88.2), turned to 180 degrees
- moved C1 62.4 mm to (42.0, 97.0), turned to 0 degrees
- moved U3 62.0 mm to (41.9, 93.6), turned to 180 degrees
- moved J1 52.6 mm to (34.1, 63.9), turned to -90 degrees
- moved U1 14.6 mm to (57.5, 72.8), turned to 180 degrees
- moved J4 5.99 mm to (81.3, 58.4)
Connections:
- net Net-(J1-In) renamed /PIN_CLOCK
- net Net-(J4-Pin_14) renamed /P2
- J4 pad 1: Net-(J4-Pin_1) -> GND
- J4 pad 10: GND -> /P0
- J4 pad 11: Net-(J4-Pin_11) -> GND
- J4 pad 12: Net-(J4-Pin_12) -> /P1
- J4 pad 13: unconnected-(J4-Pin_13-Pad13) -> GND
- J4 pad 15: Net-(J4-Pin_15) -> GND
- J4 pad 17: unconnected-(J4-Pin_17-Pad17) -> GND
- J4 pad 22: GND -> /PIN_SCK
- J4 pad 24: GND -> /PIN_RESET
- J4 pad 26: GND -> unconnected-(J4-Pin_26-Pad26)
- J4 pad 28: GND -> /PIN_SYNC
- J4 pad 29: unconnected-(J4-Pin_29-Pad29) -> GND
- J4 pad 32: GND -> unconnected-(J4-Pin_32-Pad32)
- J4 pad 5: Net-(J4-Pin_5) -> GND
- J4 pad 6: Net-(J4-Pin_6) -> unconnected-(J4-Pin_6-Pad6)
- J4 pad 7: Net-(J4-Pin_7) -> GND
- J4 pad 8: Net-(J4-Pin_8) -> GND
- J4 pad 9: Net-(J4-Pin_9) -> GND
- J5 pad 1: Net-(J5-In) -> /TRIG_IN
- U1 pad 1: unconnected-(U1-GPIO0-Pad1) -> /PIN_MISO
- U1 pad 11: Net-(J5-In) -> /PIN_UPDATE
- U1 pad 12: Net-(J4-Pin_12) -> /P3
- U1 pad 15: unconnected-(U1-GPIO11-Pad15) -> /P1
- U1 pad 16: Net-(J4-Pin_15) -> /P0
- U1 pad 19: Net-(J4-Pin_11) -> unconnected-(U1-GPIO14-Pad19)
- U1 pad 20: Net-(J4-Pin_1) -> unconnected-(U1-GPIO15-Pad20)
- U1 pad 21: Net-(J4-Pin_8) -> /TRIG_IN
- U1 pad 22: Net-(J4-Pin_7) -> unconnected-(U1-GPIO17-Pad22)
- U1 pad 24: Net-(J4-Pin_6) -> unconnected-(U1-GPIO18-Pad24)
- U1 pad 25: Net-(J4-Pin_5) -> /PIN_MOSI
- U1 pad 29: Net-(J4-Pin_9) -> unconnected-(U1-GPIO22-Pad29)
- U1 pad 33: unconnected-(U1-AGND-Pad33) -> GND
- U1 pad 5: unconnected-(U1-GPIO3-Pad5) -> /PIN_SYNC
- U1 pad 6: unconnected-(U1-GPIO4-Pad6) -> /PIN_RESET
- U1 pad 9: unconnected-(U1-GPIO6-Pad9) -> /PIN_SCK
Routing:
- net Net-(J4-Pin_12): track 92.7 -> 0.00 mm
- net Net-(J5-In): track 90.8 -> 0.00 mm
- net Net-(J4-Pin_1): track 57.5 -> 0.00 mm
- net Net-(J4-Pin_15): track 55.2 -> 0.00 mm
- net /P2: track 68.4 -> 17.4 mm
- net Net-(J4-Pin_11): track 48.7 -> 0.00 mm
- net Net-(J4-Pin_9): track 47.5 -> 0.00 mm
- net /PIN_MOSI: track 0.00 -> 45.5 mm
- net /PIN_CLOCK: track 43.7 -> 14.8 mm
- net 3V3: track 46.0 -> 21.7 mm
- net Net-(J4-Pin_8): track 19.7 -> 0.00 mm
- net Net-(J4-Pin_7): track 19.7 -> 0.00 mm
- net /TRIG_IN: track 0.00 -> 19.6 mm
- net /P0: track 0.00 -> 18.7 mm
- net Net-(J4-Pin_6): track 18.6 -> 0.00 mm
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Other:
- board size 56 x 65 mm -> 53 x 65 mm
